File: Hardware/Bottom/UknownWatch_Bottom.sch (EAGLE design)
At the start: 33 parts

Commit message: Completed take 5 and did part of take 6.
Parts:
- added C3, C5, C6: 1u, LinnesLab-Passives:CAPACITOR0603
- added C4, C7: 4.7u, LinnesLab-Passives:CAPACITOR0603
- added CHRG2: MCP73831, LinnesLab-Power:MCP73831
- added LDO2: MIC5504, LinnesLab-Power:MIC5504
- added R11: (no value), LinnesLab-Passives:RESISTOR0603
- added R12: 100k, LinnesLab-Passives:RESISTOR0603
- added U4: PCF8523, LinnesLab-Clocks:PCF8523
- added XTAL2: 32.7680kHz, LinnesLab-Clocks:CRYSTALECS-.327-12.5-12-C-TR
Connections:
- new net D27/CHRG.STATUS: CHRG2.STAT, R12.1
- new net N$1: U4.OSCI, XTAL2.2
- new net N$2: CHRG2.PROG, R11.2
- new net N$6: U4.OSCO, XTAL2.1
- new net VIN: C5.2, C7.2, CHRG2.VIN, LDO2.EN, LDO2.IN, R12.2
- new net VLIPO: C4.1, CHRG2.VBAT
- net 3.3V: now also C3.1, C6.1, LDO2.OUT, U4.VDD
- net GND: now also C3.2, C4.2, C5.1, C6.2, C7.1, CHRG2.VSS, LDO2.GND, R11.1, U4.VSS
- net SCL: now also U4.SCL
- net SDA: now also U4.SDA
Other:
- note added: "Back-up battery if desired"
- note added: "I2C Address = 0x68h"
- note added: "Power Management"
- note added: "Real-Time Clock"
