File: Hardware/Top/UnknownWatch_Top.brd (EAGLE design)
At the start: 38 x 38 mm, 62 parts, among them SW2 SWITCH.MOM, SW6 SWITCH.MOM, U2 FT231XS, U4 PCF8523, U6 NRF52832_MODULE_MDBT42

Commit message: Nearly finished routing top board
Parts:
- moved R5 49.6 mm to (9.34, 35.2)
- moved C2 46.1 mm to (8.75, 29.7)
- moved U4 46.1 mm to (7.12, 26.4)
- moved XTAL2 46.1 mm to (2.71, 27.7)
- moved R14 45.3 mm to (1.77, 19.7), turned to 90 degrees
- moved R13 44.9 mm to (3.58, 19.7), turned to 270 degrees
- moved R4 44.9 mm to (5.98, 35.2)
- moved C29 31.2 mm to (29.1, 17.2), turned to 270 degrees
- moved C28 30.6 mm to (27.6, 17.2), turned to 90 degrees
- moved XTAL4 30.4 mm to (28.2, 19.6)
- moved R11 28.1 mm to (2.51, 11.8), flipped to the bottom, turned to 180 degrees
- moved C20 26.2 mm to (7.85, 11.8), flipped to the bottom
- moved D3 25.1 mm to (8.23, -12.7)
- moved C33 25.1 mm to (8.43, -11.1)
- moved R19 25.1 mm to (8.20, -9.66)
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Routing:
- net USB-: track 1.43 -> 20.2 mm, vias 0 -> 1
- net USB+: track 1.52 -> 15.5 mm, vias 0 -> 1
- net VIN: track 7.64 -> 17.1 mm
- net GND: track 42.4 -> 51.6 mm, vias 11 -> 14
- net VLIPO: track 14.1 -> 21.0 mm
- net N$17: track 0.00 -> 6.64 mm
- net N$27: track 0.00 -> 4.13 mm
- net N$26: track 0.00 -> 3.83 mm
- net N$2: track 6.11 -> 2.34 mm
- net N$13: track 4.53 -> 2.26 mm
- net A4/BATT: track 0.00 -> 1.83 mm

Commit message: Completed take 5 and did part of take 6.
Parts:
- removed C2, C5, C6: 1u, LinnesLab-Passives:C0603
- removed C20, C21: 4.7u, LinnesLab-Passives:C0603
- removed CHRG2: MCP73831, LinnesLab-Power:SOT23-5
- removed LDO2: MIC5504, LinnesLab-Power:SOT23-5
- removed R11: (no value), LinnesLab-Passives:R0603
- removed R12: 100k, LinnesLab-Passives:R0603
- removed SD2: (no value), LinnesLab-Connectors:MICROSD
- removed U4: PCF8523, LinnesLab-Clocks:SO8
- removed XTAL2: 32.7680kHz, LinnesLab-Clocks:2-SMD.NOLEAD.2.0MMTO1.2MM
- moved SW8 40.7 mm to (32.6, 17.6)
- moved D3 35.8 mm to (33.2, 12.9), turned to 180 degrees
- moved R19 35.2 mm to (33.4, 15.0), turned to 180 degrees
- moved C33 33.6 mm to (33.6, 11.1), turned to 0 degrees
- moved LED6 18.9 mm to (34.2, 20.8), turned to 270 degrees
- moved LED5 18.5 mm to (32.1, 20.9), turned to 270 degrees
- moved SW7 17.2 mm to (34.6, 35.6)
- moved C29 14.2 mm to (16.3, 23.5), turned to 180 degrees
- moved R18 14.0 mm to (34.2, 24.2), turned to 90 degrees
- moved R17 13.6 mm to (32.1, 24.2), turned to 90 degrees
- moved CORTEX3 13.4 mm to (34.7, 29.7), turned to 270 degrees
- moved C28 12.3 mm to (16.2, 21.8), turned to 0 degrees
- moved SW6 10.4 mm to (21.8, 4.51), turned to 180 degrees
- moved C32 10.0 mm to (14.8, 27.3), turned to 270 degrees
- moved SW2 9.98 mm to (32.2, 4.64), turned to 180 degrees
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Connections:
- removed net CD2: SD2.CD2
- removed net N$17: CHRG2.5, R11.2
- removed net N$6: U4.2, XTAL2.P$1
- removed net N$9: U4.1, XTAL2.P$2
- removed net VBAT: U4.3
- net 3.3V: no longer C2.1, C6.1, LDO2.5, SD2.4, U4.8
- net D27/CHRG.STATUS: no longer CHRG2.1, R12.1
- net D5/CD1: no longer SD2.CD1
- net D7/SD.CS: no longer SD2.2
- net GND: no longer C2.2, C20.2, C21.1, C5.1, C6.2, CHRG2.2, LDO2.2, R11.1, SD2.6, SD2.MT1, SD2.MT2, U4.4
- net MISO: no longer SD2.7
- net MOSI: no longer SD2.3
- net SCK: no longer SD2.5
- net SCL: no longer U4.6
- net SDA: no longer U4.5
- net VIN: no longer C21.2, C5.2, CHRG2.4, LDO2.1, LDO2.3, R12.2
- net VLIPO: no longer C20.1, CHRG2.3
Routing:
- net RESET: track 0.00 -> 28.1 mm, vias 0 -> 1
- net D15/SW2: track 0.00 -> 25.3 mm
- net DTR: track 0.00 -> 24.2 mm, vias 0 -> 2
- net D16/CS.OLED: track 0.00 -> 22.4 mm, vias 0 -> 2
- net D11/SW1: track 0.00 -> 18.6 mm
- net SCK: track 0.00 -> 18.1 mm, vias 0 -> 2
- net MOSI: track 0.00 -> 16.3 mm, vias 0 -> 2
- net D4/DC.OLED: track 0.00 -> 15.0 mm, vias 0 -> 2
- net SWO: track 0.00 -> 13.7 mm, vias 0 -> 1
- net D3/RESET.OLED: track 0.00 -> 11.5 mm
- net VIN: track 17.1 -> 6.27 mm
- net DFU: track 0.00 -> 9.91 mm, vias 0 -> 2
- net SWCLK: track 0.00 -> 9.71 mm
- net N$17: track 6.64 -> 0.00 mm
- net SWDIO: track 0.00 -> 6.43 mm, vias 0 -> 1
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